File: BSE_Comparator.kicad_sch (KiCad schematic)
At the start: 4 parts, among them U4 LM393, U5 74AHC1G32

Commit message: completed initial schematic
Parts:
- U4: footprint (none) -> Package_SO:SOIC-8-N7_3.9x4.9mm_P1.27mm
- U5: footprint (none) -> Package_TO_SOT_SMD:SOT-353_SC-70-5
Changed lines of the file:
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@@
       (effects (font (size 1.27 1.27)) (justify left))
     )
-    (property "Footprint" "" (id 2) (at 90.17 100.33 0)
+    (property "Footprint" "Package_SO:SOIC-8-N7_3.9x4.9mm_P1.27mm" (id 2) (at 90.17 100.33 0)
       (effects (font (size 1.27 1.27)) hide)
     )
@@
     (property "Reference" "U4" (id 0) (at 146.05 75.0402 0))
     (property "Value" "LM393" (id 1) (at 146.05 77.5771 0))
-    (property "Footprint" "" (id 2) (at 146.05 83.82 0)
+    (property "Footprint" "Package_SO:SOIC-8-N7_3.9x4.9mm_P1.27mm" (id 2) (at 146.05 83.82 0)
       (effects (font (size 1.27 1.27)) hide)
     )
@@
     (property "Reference" "U5" (id 0) (at 173.355 89.7636 0))
     (property "Value" "74AHC1G32" (id 1) (at 173.355 92.075 0))
-    (property "Footprint" "" (id 2) (at 166.37 95.25 0)
+    (property "Footprint" "Package_TO_SOT_SMD:SOT-353_SC-70-5" (id 2) (at 166.37 95.25 0)
       (effects (font (size 1.27 1.27)) hide)
     )
@@
     (property "Reference" "U4" (id 0) (at 146.05 97.9002 0))
     (property "Value" "LM393" (id 1) (at 146.05 100.4371 0))
-    (property "Footprint" "" (id 2) (at 146.05 106.68 0)
+    (property "Footprint" "Package_SO:SOIC-8-N7_3.9x4.9mm_P1.27mm" (id 2) (at 146.05 106.68 0)
       (effects (font (size 1.27 1.27)) hide)
     )

Commit message: post revision 1
Parts:
- removed U5: 74AHC1G32, Package_TO_SOT_SMD:SOT-353_SC-70-5, symbol 74xGxx:74AHC1G32
- added D10, D7, D8, D9: D_Small, Diode_SMD:D_SMC, symbol Device:D_Small
- added R24: 3k, Resistor_SMD:R_0603_1608Metric, symbol Device:R_Small
- renumbered U4 to U5
Connections:
- net +5V: now also D7.1 (K), D9.1 (K); no longer RV1.1, RV2.1
- net Brake: now also U5.1, U5.7, R24.2
- net Brake1: now also D7.2 (A), D8.1 (K)
- net Brake2: now also D10.1 (K), D9.2 (A)
- net GND: now also D10.2 (A), D8.2 (A), R24.1
- new net +3V3: RV1.1, RV2.1
Other:
- moved on the sheet: RV1, RV2, U5A, U5B, U5C
