File: BSE_Comparator.kicad_sch (KiCad schematic)
At the start: 6 parts, among them U4 LM393

Commit message: layout
Parts:
- U4: footprint Package_SO:SOIC-8-N7_3.9x4.9mm_P1.27mm -> Package_SO:SOIC-8_3.9x4.9mm_P1.27mm
Changed lines of the file:
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@@
       (effects (font (size 1.27 1.27)) (justify left))
     )
-    (property "Footprint" "Package_SO:SOIC-8-N7_3.9x4.9mm_P1.27mm" (id 2) (at 120.65 97.79 0)
+    (property "Footprint" "Package_SO:SOIC-8_3.9x4.9mm_P1.27mm" (id 2) (at 120.65 97.79 0)
       (effects (font (size 1.27 1.27)) hide)
     )
@@
     (property "Reference" "U4" (id 0) (at 175.26 75.0402 0))
     (property "Value" "LM393" (id 1) (at 175.26 77.5771 0))
-    (property "Footprint" "Package_SO:SOIC-8-N7_3.9x4.9mm_P1.27mm" (id 2) (at 175.26 83.82 0)
+    (property "Footprint" "Package_SO:SOIC-8_3.9x4.9mm_P1.27mm" (id 2) (at 175.26 83.82 0)
       (effects (font (size 1.27 1.27)) hide)
     )
@@
     (pin "4")
     (pin "8")
-  )
-  (symbol (lib_id "power:+3V3") (at 149.86 115.57 0) (unit 1)
-    (in_bom yes) (on_board yes) (fields_autoplaced)
-    (property "Reference" "#PWR056" (id 0) (at 149.86 119.38 0)
-      (effects (font (size 1.27 1.27)) hide)
-    )
-    (property "Value" "+3V3" (id 1) (at 149.86 111.9942 0))
-    (property "Footprint" "" (id 2) (at 149.86 115.57 0)
-      (effects (font (size 1.27 1.27)) hide)
-    )
-    (property "Datasheet" "" (id 3) (at 149.86 115.57 0)
-      (effects (font (size 1.27 1.27)) hide)
-    )
-    (pin "1")
   )
   (symbol (lib_id "Device:R_Potentiometer_Trim") (at 149.86 91.44 0) (unit 1)
@@
     (property "Reference" "U4" (id 0) (at 175.26 102.9802 0))
     (property "Value" "LM393" (id 1) (at 175.26 105.5171 0))
-    (property "Footprint" "Package_SO:SOIC-8-N7_3.9x4.9mm_P1.27mm" (id 2) (at 175.26 111.76 0)
+    (property "Footprint" "Package_SO:SOIC-8_3.9x4.9mm_P1.27mm" (id 2) (at 175.26 111.76 0)
       (effects (font (size 1.27 1.27)) hide)
     )
@@
     (pin "1")
   )
+  (symbol (lib_id "power:+3V3") (at 149.86 115.57 0) (unit 1)
+    (in_bom yes) (on_board yes) (fields_autoplaced)
+    (property "Reference" "#PWR?" (id 0) (at 149.86 119.38 0)
+      (effects (font (size 1.27 1.27)) hide)
+    )
+    (property "Value" "+3V3" (id 1) (at 149.86 111.9942 0))
+    (property "Footprint" "" (id 2) (at 149.86 115.57 0)
+      (effects (font (size 1.27 1.27)) hide)
+    )
+    (property "Datasheet" "" (id 3) (at 149.86 115.57 0)
+      (effects (font (size 1.27 1.27)) hide)
+    )
+    (pin "1")
+  )
   (symbol (lib_id "power:+3V3") (at 149.86 87.63 0) (unit 1)
     (in_bom yes) (on_board yes) (fields_autoplaced)
-    (property "Reference" "#PWR054" (id 0) (at 149.86 91.44 0)
+    (property "Reference" "#PWR?" (id 0) (at 149.86 91.44 0)
       (effects (font (size 1.27 1.27)) hide)
     )
