File: Brake_Light.kicad_sch (KiCad schematic)
At the start: 9 parts, among them J1 Conn_01x06, J2 Conn_01x02, Q1 AO3400A, U1 LM317_TO-252

Commit message: finalized
Parts:
- removed C1: 100n, Capacitor_SMD:C_0603_1608Metric, symbol Device:C_Small
- removed C2: 1u, Capacitor_SMD:C_0603_1608Metric, symbol Device:C_Small
- removed U1: LM317_TO-252, Package_TO_SOT_SMD:TO-252-2, symbol Regulator_Linear:LM317_TO-252
- R1: value 1.1k -> 2k; footprint Resistor_SMD:R_0603_1608Metric -> (none)
- R2: value 10k -> 1k5; footprint Resistor_SMD:R_0603_1608Metric -> (none)
Connections:
- net Brake_Output: now also R1.1
- net GND: now also R2.2; no longer R1.2
- net at Q1.1 (G), R2.1: now also R1.2
Other:
- moved on the sheet: J2, Q1, R3

Commit message: layout
Parts:
- removed R3: 10k, Resistor_SMD:R_0603_1608Metric, symbol Device:R_Small
- R1, R2: footprint (none) -> Resistor_SMD:R_0603_1608Metric
Connections:
- net +12V is gone; now on net +24V: Q1.3 (D)
- net at Q1.2 (S): now also J2.1 (Pin_1)
Changed lines of the file:
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@@
     (stroke (width 0) (type default) (color 0 0 0 0))
   )
-  (wire (pts (xy 82.55 152.4) (xy 82.55 153.67))
+  (wire (pts (xy 82.55 147.32) (xy 82.55 153.67))
     (stroke (width 0) (type default) (color 0 0 0 0))
   )
@@
     (pin "1")
   )
+  (symbol (lib_id "power:+24V") (at 82.55 137.16 0) (unit 1)
+    (in_bom yes) (on_board yes) (fields_autoplaced)
+    (property "Reference" "#PWR0101" (id 0) (at 82.55 140.97 0)
+      (effects (font (size 1.27 1.27)) hide)
+    )
+    (property "Value" "+24V" (id 1) (at 82.55 133.5842 0))
+    (property "Footprint" "" (id 2) (at 82.55 137.16 0)
+      (effects (font (size 1.27 1.27)) hide)
+    )
+    (property "Datasheet" "" (id 3) (at 82.55 137.16 0)
+      (effects (font (size 1.27 1.27)) hide)
+    )
+    (pin "1")
+  )
   (symbol (lib_id "Transistor_FET:AO3400A") (at 80.01 142.24 0) (unit 1)
     (in_bom yes) (on_board yes) (fields_autoplaced)
@@
     )
     (property "Datasheet" "" (id 3) (at 86.36 157.48 0)
-      (effects (font (size 1.27 1.27)) hide)
-    )
-    (pin "1")
-  )
-  (symbol (lib_id "power:+12V") (at 82.55 137.16 0) (unit 1)
-    (in_bom yes) (on_board yes) (fields_autoplaced)
-    (property "Reference" "#PWR04" (id 0) (at 82.55 140.97 0)
-      (effects (font (size 1.27 1.27)) hide)
-    )
-    (property "Value" "+12V" (id 1) (at 82.55 133.5842 0))
-    (property "Footprint" "" (id 2) (at 82.55 137.16 0)
-      (effects (font (size 1.27 1.27)) hide)
-    )
-    (property "Datasheet" "" (id 3) (at 82.55 137.16 0)
       (effects (font (size 1.27 1.27)) hide)
     )
@@
       (effects (font (size 1.27 1.27)) (justify left))
     )
-    (property "Footprint" "" (id 2) (at 71.12 137.16 0)
+    (property "Footprint" "Resistor_SMD:R_0603_1608Metric" (id 2) (at 71.12 137.16 0)
       (effects (font (size 1.27 1.27)) hide)
     )
@@
       (effects (font (size 1.27 1.27)) (justify left))
     )
-    (property "Footprint" "" (id 2) (at 71.12 147.32 0)
+    (property "Footprint" "Resistor_SMD:R_0603_1608Metric" (id 2) (at 71.12 147.32 0)
       (effects (font (size 1.27 1.27)) hide)
     )
@@
     )
     (pin "1")
-  )
-  (symbol (lib_id "Device:R_Small") (at 82.55 149.86 0) (unit 1)
-    (in_bom yes) (on_board yes)
-    (property "Reference" "R3" (id 0) (at 83.82 149.86 0)
-      (effects (font (size 1.27 1.27)) (justify left))
-    )
-    (property "Value" "10k" (id 1) (at 77.47 149.86 0)
-      (effects (font (size 1.27 1.27)) (justify left))
-    )
-    (property "Footprint" "Resistor_SMD:R_0603_1608Metric" (id 2) (at 82.55 149.86 0)
-      (effects (font (size 1.27 1.27)) hide)
-    )
-    (property "Datasheet" "~" (id 3) (at 82.55 149.86 0)
-      (effects (font (size 1.27 1.27)) hide)
-    )
-    (pin "1")
-    (pin "2")
   )
   (symbol (lib_id "power:GND") (at 71.12 149.86 0) (unit 1)
@@
       (reference "#PWR03") (unit 1) (value "GND") (footprint "")
     )
-    (path "/7a9b31f6-7595-47cf-a050-1ae8cfca436e"
-      (reference "#PWR04") (unit 1) (value "+12V") (footprint "")
-    )
     (path "/76196397-99a2-41c3-86bb-f323bd352b60"
       (reference "#PWR05") (unit 1) (value "GND") (footprint "")
@@
       (reference "#PWR053") (unit 1) (value "GND") (footprint "")
     )
-    (path "/599b7a84-d6d4-475d-aa4b-696e962196c6/e3d4b6f4-7568-4362-a6f5-e771c20073a3"
-      (reference "#PWR054") (unit 1) (value "+3V3") (footprint "")
-    )
     (path "/599b7a84-d6d4-475d-aa4b-696e962196c6/afbf2d05-fe67-4c2e-a005-9c54d1179aaa"
       (reference "#PWR055") (unit 1) (value "GND") (footprint "")
     )
-    (path "/599b7a84-d6d4-475d-aa4b-696e962196c6/89f96146-3093-4e58-9926-55f2523468b9"
-      (reference "#PWR056") (unit 1) (value "+3V3") (footprint "")
-    )
     (path "/599b7a84-d6d4-475d-aa4b-696e962196c6/7e6b00cf-9689-4efe-962f-92dbaa1d217b"
       (reference "#PWR057") (unit 1) (value "GND") (footprint "")
@@
       (reference "#PWR067") (unit 1) (value "GND") (footprint "")
     )
+    (path "/517b2523-0ed7-47ce-96b0-62547732ef64"
+      (reference "#PWR0101") (unit 1) (value "+24V") (footprint "")
+    )
+    (path "/599b7a84-d6d4-475d-aa4b-696e962196c6/e311d513-65d4-4ab1-9091-8e7ff9217008"
+      (reference "#PWR?") (unit 1) (value "+3V3") (footprint "")
+    )
+    (path "/599b7a84-d6d4-475d-aa4b-696e962196c6/f323bd76-41aa-4d9e-8b8f-c99d6a6502ef"
+      (reference "#PWR?") (unit 1) (value "+3V3") (footprint "")
+    )
     (path "/29639228-78f8-4f5b-8652-d63c64ba8913/00000000-0000-0000-0000-00006343a469"
       (reference "C1") (unit 1) (value "4u7") (footprint "Capacitor_SMD:C_0603_1608Metric")
@@
     )
     (path "/29639228-78f8-4f5b-8652-d63c64ba8913/03bb6952-8654-4c84-bec4-48dc9118f988"
-      (reference "D2") (unit 1) (value "DT1446-04TS-7") (footprint "SOT95P280X100-6N")
+      (reference "D2") (unit 1) (value "DT1446-04TS-7") (footprint "Global Libraries:SOT95P280X100-6N")
     )
     (path "/29639228-78f8-4f5b-8652-d63c64ba8913/96af04c7-0dd8-4324-89bc-82ee00f61136"
@@
     )
     (path "/ace78a4d-9441-4350-b054-4de2210fc7c9"
-      (reference "R1") (unit 1) (value "2k") (footprint "")
+      (reference "R1") (unit 1) (value "2k") (footprint "Resistor_SMD:R_0603_1608Metric")
     )
     (path "/bd15a47c-4079-4b6b-8d0b-d9ac69731a22"
-      (reference "R2") (unit 1) (value "1k5") (footprint "")
-    )
-    (path "/cd6f1af6-5e59-489a-90ef-46e1edd90692"
-      (reference "R3") (unit 1) (value "10k") (footprint "Resistor_SMD:R_0603_1608Metric")
+      (reference "R2") (unit 1) (value "1k5") (footprint "Resistor_SMD:R_0603_1608Metric")
     )
     (path "/29639228-78f8-4f5b-8652-d63c64ba8913/00000000-0000-0000-0000-00006353dea1"
@@
     )
     (path "/599b7a84-d6d4-475d-aa4b-696e962196c6/87cb97e9-836e-4fb8-8473-bf8302a52584"
-      (reference "U4") (unit 1) (value "LM393") (footprint "Package_SO:SOIC-8-N7_3.9x4.9mm_P1.27mm")
+      (reference "U4") (unit 1) (value "LM393") (footprint "Package_SO:SOIC-8_3.9x4.9mm_P1.27mm")
     )
     (path "/599b7a84-d6d4-475d-aa4b-696e962196c6/c5177256-8ac6-4beb-b6f6-fbb4e57619be"
-      (reference "U4") (unit 2) (value "LM393") (footprint "Package_SO:SOIC-8-N7_3.9x4.9mm_P1.27mm")
+      (reference "U4") (unit 2) (value "LM393") (footprint "Package_SO:SOIC-8_3.9x4.9mm_P1.27mm")
     )
     (path "/599b7a84-d6d4-475d-aa4b-696e962196c6/6a89753f-d7ff-4b02-9da8-c831b305bced"
-      (reference "U4") (unit 3) (value "LM393") (footprint "Package_SO:SOIC-8-N7_3.9x4.9mm_P1.27mm")
+      (reference "U4") (unit 3) (value "LM393") (footprint "Package_SO:SOIC-8_3.9x4.9mm_P1.27mm")
     )
     (path "/4b3960a9-3979-4ced-9a60-8a8791847dc9/5eef7685-46e3-4490-b1c3-d367d5bf00e5/8cd40687-f12d-4487-81ad-e4b3943431ac"
