File: Brake_Light.kicad_pcb (KiCad board)
At the start: 2 copper layers, 76.2 x 50.8 mm, 87 parts, among them J1 Conn_01x06, J2 Conn_01x02, J3 Conn_01x02, J4 Conn_01x02, J5 SWD, Q1 AO3400A, SW1 SW_SPDT, U1 STM32F105RCTx, U2 SN65HVD230, U3 SN65HVD230, U4 LM393, U5 LMR51420, U6 AMS1117-3.3, Y1 16MHz

Commit message: finished layout
Parts:
- added  : LOGO, LOGO, B.Cu at (119.9, 65.3)
Routing:
- net +3.3V: track 101.0 -> 145.1 mm, vias 4 -> 14
- net /Brake_Signal: track 7.51 -> 36.4 mm, vias 0 -> 2
- net +5V: track 96.6 -> 107.6 mm, vias 6 -> 8
- net GND: track 183.3 -> 190.2 mm, vias 18 -> 21
- net /Microcontroller/CAN1_RX: track 34.5 -> 38.2 mm
- net /StandardizedVRMS/BUCK/V_in: track 63.8 -> 66.7 mm
- net /Brake_Output: track 53.8 -> 55.7 mm
- net Net-(J2-Pad1): track 12.9 -> 14.7 mm
- net Net-(D2-Pad1): track 21.8 -> 22.9 mm
- net /Brake2: track 23.1 -> 24.2 mm
- net /Brake1: track 23.4 -> 24.2 mm
- net +24V: track 26.7 -> 27.5 mm
- net Net-(RV1-Pad2): track 19.2 -> 20.0 mm
- net /Microcontroller/SWDIO: track 62.7 -> 63.3 mm
Other:
- board size 76.2 x 50.8 mm -> 55.1 x 41.8 mm
- board text added: "Brake Light Controller"
- board text added: "Sahil Shah"
